Commit message: finished my robotic arm assignment

File: Task4solution/task4workspace/install/kuka_description/share/kuka_description/urdf/kuka.urdf (robot description, URDF)
Before this commit: robot dogg, 1 links, 0 joints
Links:
- link base_link: geometry visual mesh filename=package://kuka_description/meshes/link_0.dae scale=1.0 1.0 1.0
